File: NekoESC_V1/ESC.kicad_sch (KiCad schematic)
At the start: 33 parts, among them Q201 NMOS, Q202 NMOS, Q203 NMOS, Q204 NMOS, Q205 NMOS, Q206 NMOS, U201 GD32E230G8U6, U202 FD6288Q

Commit message: add c1206
Parts:
- Q201, Q202, Q203, Q204, Q205, Q206: footprint myLib:DFN8_3x3_MOS_GSD -> SMTOPT:DFN-8_3x3_MOS_GSD
Changed lines of the file:
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@@
 			)
 		)
-		(property "Footprint" "myLib:DFN8_3x3_MOS_GSD"
+		(property "Footprint" "SMTOPT:DFN-8_3x3_MOS_GSD"
 			(at 158.75 41.91 0)
 			(effects
@@
 			)
 		)
-		(property "Footprint" "myLib:DFN8_3x3_MOS_GSD"
+		(property "Footprint" "SMTOPT:DFN-8_3x3_MOS_GSD"
 			(at 212.09 41.91 0)
 			(effects
@@
 			)
 		)
-		(property "Footprint" "myLib:DFN8_3x3_MOS_GSD"
+		(property "Footprint" "SMTOPT:DFN-8_3x3_MOS_GSD"
 			(at 158.75 57.15 0)
 			(effects
@@
 			)
 		)
-		(property "Footprint" "myLib:DFN8_3x3_MOS_GSD"
+		(property "Footprint" "SMTOPT:DFN-8_3x3_MOS_GSD"
 			(at 264.16 57.15 0)
 			(effects
@@
 			)
 		)
-		(property "Footprint" "myLib:DFN8_3x3_MOS_GSD"
+		(property "Footprint" "SMTOPT:DFN-8_3x3_MOS_GSD"
 			(at 212.09 57.15 0)
 			(effects
@@
 			)
 		)
-		(property "Footprint" "myLib:DFN8_3x3_MOS_GSD"
+		(property "Footprint" "SMTOPT:DFN-8_3x3_MOS_GSD"
 			(at 264.16 41.91 0)
 			(effects

Commit message: update lib
Parts:
- U201: footprint Package_DFN_QFN:WQFN-28-1EP_4x4mm_P0.4mm_EP2.7x2.7mm -> SMTOPT:WQFN-28-1EP_4x4mm_P0.4mm_EP2.7x2.7mm
- U202: footprint Package_DFN_QFN:QFN-24-1EP_4x4mm_P0.5mm_EP2.7x2.7mm -> SMTOPT:QFN-24-1EP_4x4mm_P0.5mm_EP2.7x2.7mm
Changed lines of the file:
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@@
 			)
 		)
-		(property "Footprint" "Package_DFN_QFN:WQFN-28-1EP_4x4mm_P0.4mm_EP2.7x2.7mm"
+		(property "Footprint" "SMTOPT:WQFN-28-1EP_4x4mm_P0.4mm_EP2.7x2.7mm"
 			(at 82.55 35.56 0)
 			(effects
@@
 			)
 		)
-		(property "Footprint" "Package_DFN_QFN:QFN-24-1EP_4x4mm_P0.5mm_EP2.7x2.7mm"
+		(property "Footprint" "SMTOPT:QFN-24-1EP_4x4mm_P0.5mm_EP2.7x2.7mm"
 			(at 121.92 116.84 0)
 			(effects

Commit message: modify hardware
Parts:
- R217: value 1K -> 10K
Connections:
- net +3V3: now also R217.1
- net GND: now also U201.1 (BOOT0); no longer R217.2
- net NRST: now also R217.2
- removed net BOOT: R217.1, U201.1 (BOOT0)
Changed lines of the file:
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@@
 		)
 	)
-	(label "BOOT"
-		(at 58.42 50.8 0)
-		(effects
-			(font
-				(size 1.27 1.27)
-			)
-			(justify left bottom)
-		)
-	)
 	(label "HO_B1"
 		(at 187.96 44.45 0)
@@
 	(symbol
 		(lib_id "Device:R")
+		(at 40.64 81.28 0)
+		(unit 1)
+		(exclude_from_sim no)
+		(in_bom yes)
+		(on_board yes)
+		(dnp no)
+		(fields_autoplaced yes)
+		(property "Reference" "R217"
+			(at 43.18 80.0099 0)
+			(effects
+				(font
+					(size 1.27 1.27)
+				)
+				(justify left)
+			)
+		)
+		(property "Value" "10K"
+			(at 43.18 82.5499 0)
+			(effects
+				(font
+					(size 1.27 1.27)
+				)
+				(justify left)
+			)
+		)
+		(property "Footprint" "SMTOPT:R_0402"
+			(at 38.862 81.28 90)
+			(effects
+				(font
+					(size 1.27 1.27)
+				)
+				(hide yes)
+			)
+		)
+		(property "Datasheet" "~"
+			(at 40.64 81.28 0)
+			(effects
+				(font
+					(size 1.27 1.27)
+				)
+				(hide yes)
+			)
+		)
+		(property "Description" "Resistor"
+			(at 40.64 81.28 0)
+			(effects
+				(font
+					(size 1.27 1.27)
+				)
+				(hide yes)
+			)
+		)
+		(pin "2"
+		)
+		(pin "1"
+		)
+		(instances
+			(project "NekoESC"
+				(path "/8f4d8a7b-a7cd-45c1-8128-94732b967d72/01eec08a-f765-4872-84ac-8ff7479be631"
+					(reference "R219")
+					(unit 1)
+				)
+				(path "/8f4d8a7b-a7cd-45c1-8128-94732b967d72/4325d277-4d64-41a1-9c1c-720f24911c6a"
+					(reference "R218")
+					(unit 1)
+				)
+				(path "/8f4d8a7b-a7cd-45c1-8128-94732b967d72/8dde3b75-bc2c-4ba6-9104-f13124f553da"
+					(reference "R220")
+					(unit 1)
+				)
+				(path "/8f4d8a7b-a7cd-45c1-8128-94732b967d72/c34570e9-2a74-4c8d-9ad9-a9577ddad226"
+					(reference "R217")
+					(unit 1)
+				)
+			)
+		)
+	)
+	(symbol
+		(lib_id "Device:R")
 		(at 180.34 115.57 270)
 		(unit 1)
@@
 	(symbol
 		(lib_id "power:GND")
-		(at 50.8 50.8 270)
+		(at 58.42 50.8 270)
 		(unit 1)
 		(exclude_from_sim no)
@@
 		(fields_autoplaced yes)
 		(property "Reference" "#PWR0277"
-			(at 44.45 50.8 0)
+			(at 52.07 50.8 0)
 			(effects
 				(font
@@
 		)
 		(property "Value" "GND"
-			(at 46.99 50.7999 90)
+			(at 54.61 50.7999 90)
 			(effects
 				(font
@@
 		)
 		(property "Footprint" ""
-			(at 50.8 50.8 0)
+			(at 58.42 50.8 0)
 			(effects
 				(font
@@
 		)
 		(property "Datasheet" ""
-			(at 50.8 50.8 0)
+			(at 58.42 50.8 0)
 			(effects
 				(font
@@
 		)
 		(property "Description" "Power symbol creates a global label with name \"GND\" , ground"
-			(at 50.8 50.8 0)
+			(at 58.42 50.8 0)
 			(effects
 				(font
@@
 	)
 	(symbol
-		(lib_id "Device:R")
-		(at 54.61 50.8 270)
+		(lib_id "Device:D_Schottky")
+		(at 135.89 31.75 180)
 		(unit 1)
 		(exclude_from_sim no)
@@
 		(dnp no)
 		(fields_autoplaced yes)
-		(property "Reference" "R217"
-			(at 54.61 44.45 90)
+		(property "Reference" "D201"
+			(at 136.2075 25.4 0)
 			(effects
 				(font
@@
 			)
 		)
-		(property "Value" "1K"
-			(at 54.61 46.99 90)
+		(property "Value" "1N5819"
+			(at 136.2075 27.94 0)
 			(effects
 				(font
@@
 			)
 		)
-		(property "Footprint" "SMTOPT:R_0402"
-			(at 54.61 49.022 90)
+		(property "Footprint" "SMTOPT:D_SOD-323"
+			(at 135.89 31.75 0)
 			(effects
 				(font
@@
 		)
 		(property "Datasheet" "~"
-			(at 54.61 50.8 0)
+			(at 135.89 31.75 0)
 			(effects
 				(font
@@
 			)
 		)
-		(property "Description" "Resistor"
-			(at 54.61 50.8 0)
+		(property "Description" "Schottky diode"
+			(at 135.89 31.75 0)
 			(effects
 				(font
@@
 		)
 		(instances
-			(project "NekoESC"
+			(project "NekoFC_AIO"
 				(path "/8f4d8a7b-a7cd-45c1-8128-94732b967d72/01eec08a-f765-4872-84ac-8ff7479be631"
-					(reference "R219")
+					(reference "D401")
 					(unit 1)
 				)
 				(path "/8f4d8a7b-a7cd-45c1-8128-94732b967d72/4325d277-4d64-41a1-9c1c-720f24911c6a"
-					(reference "R218")
+					(reference "D301")
 					(unit 1)
 				)
 				(path "/8f4d8a7b-a7cd-45c1-8128-94732b967d72/8dde3b75-bc2c-4ba6-9104-f13124f553da"
-					(reference "R220")
+					(reference "D501")
 					(unit 1)
 				)
 				(path "/8f4d8a7b-a7cd-45c1-8128-94732b967d72/c34570e9-2a74-4c8d-9ad9-a9577ddad226"
-					(reference "R217")
+					(reference "D201")
 					(unit 1)
 				)
@@
 	)
 	(symbol
-		(lib_id "Device:D_Schottky")
-		(at 135.89 31.75 180)
+		(lib_id "power:+3V3")
+		(at 40.64 77.47 0)
 		(unit 1)
 		(exclude_from_sim no)
@@
 		(dnp no)
 		(fields_autoplaced yes)
-		(property "Reference" "D201"
-			(at 136.2075 25.4 0)
+		(property "Reference" "#PWR0278"
+			(at 40.64 81.28 0)
 			(effects
 				(font
 					(size 1.27 1.27)
 				)
+				(hide yes)
 			)
 		)
-		(property "Value" "1N5819"
-			(at 136.2075 27.94 0)
+		(property "Value" "+3V3"
+			(at 40.64 72.39 0)
 			(effects
 				(font
@@
 			)
 		)
-		(property "Footprint" "SMTOPT:D_SOD-323"
-			(at 135.89 31.75 0)
+		(property "Footprint" ""
+			(at 40.64 77.47 0)
 			(effects
 				(font
@@
 			)
 		)
-		(property "Datasheet" "~"
-			(at 135.89 31.75 0)
+		(property "Datasheet" ""
+			(at 40.64 77.47 0)
 			(effects
 				(font
@@
 			)
 		)
-		(property "Description" "Schottky diode"
-			(at 135.89 31.75 0)
+		(property "Description" "Power symbol creates a global label with name \"+3V3\""
+			(at 40.64 77.47 0)
 			(effects
 				(font
@@
 			)
 		)
-		(pin "2"
-		)
 		(pin "1"
 		)
 		(instances
-			(project "NekoFC_AIO"
+			(project "NekoESC"
 				(path "/8f4d8a7b-a7cd-45c1-8128-94732b967d72/01eec08a-f765-4872-84ac-8ff7479be631"
-					(reference "D401")
+					(reference "#PWR0297")
 					(unit 1)
 				)
 				(path "/8f4d8a7b-a7cd-45c1-8128-94732b967d72/4325d277-4d64-41a1-9c1c-720f24911c6a"
-					(reference "D301")
+					(reference "#PWR0296")
 					(unit 1)
 				)
 				(path "/8f4d8a7b-a7cd-45c1-8128-94732b967d72/8dde3b75-bc2c-4ba6-9104-f13124f553da"
-					(reference "D501")
+					(reference "#PWR0298")
 					(unit 1)
 				)
 				(path "/8f4d8a7b-a7cd-45c1-8128-94732b967d72/c34570e9-2a74-4c8d-9ad9-a9577ddad226"
-					(reference "D201")
+					(reference "#PWR0278")
 					(unit 1)
 				)
