File: NekoESC_V1/NekoESC.kicad_pcb (KiCad board)
At the start: 4 copper layers, 38.5 x 38.5 mm, 194 parts, among them J101 SWD, J102 SWD, J107 JST-SH_8P, Q201 NMOS, Q202 NMOS, Q203 NMOS, Q204 NMOS, Q205 NMOS, Q206 NMOS, Q301 NMOS, Q302 NMOS, Q303 NMOS, Q304 NMOS, Q305 NMOS, Q306 NMOS, Q401 NMOS, Q402 NMOS, Q403 NMOS, Q404 NMOS, Q405 NMOS, Q406 NMOS, Q501 NMOS, Q502 NMOS, Q503 NMOS, Q504 NMOS, Q505 NMOS, Q506 NMOS, U102 ME3121, U103 INA180A1, U104 HT7533-1-SOT89, U201 GD32E230G8U6, U202 FD6288Q, U301 GD32E230G8U6, U302 FD6288Q, U401 GD32E230G8U6, U402 FD6288Q, U501 GD32E230G8U6, U502 FD6288Q

Commit message: add c1206
Parts:
- C122, C123, C124, C125, C126, C127, C128, C129, C130, C131, C133, C134, C135, C136, C138, C139, C140, C141, C142, C143, C144, C145, C146, C147, C148, C149, C150, C151, C152, C153, C154, C155, C156, C157, C158, C159, C160, C161, C162, C163: footprint Capacitor_SMD:C_1206_3216Metric -> SMTOPT:C_1206
- Q201, Q202, Q203, Q204, Q205, Q206, Q301, Q302, Q303, Q304, Q305, Q306, Q401, Q402, Q403, Q404, Q405, Q406, Q501, Q502, Q503, Q504, Q505, Q506: footprint myLib:DFN8_3x3_MOS_GSD -> SMTOPT:DFN-8_3x3_MOS_GSD

Commit message: smaller
Parts:
- removed C122, C123, C124, C125, C126, C127, C128, C129, C130, C131, C133, C135, C148, C150, C152, C154, C156, C158, C160, C162: 10uF/50V, SMTOPT:C_1206
- moved Q201 2.60 mm to (103.6, 106.0)
- moved Q202 2.60 mm to (103.6, 109.6)
- moved Q203 2.60 mm to (103.6, 113.2)
- moved Q301 2.60 mm to (103.6, 116.8)
- moved Q302 2.60 mm to (103.6, 120.4)
- moved Q303 2.60 mm to (103.6, 124.0)
Routing:
- net Net-(Q302-G): track 18.1 -> 6.46 mm, vias 2 -> 1
- net Net-(Q301-G): track 16.1 -> 5.62 mm, vias 2 -> 1
- net Net-(Q203-G): track 18.9 -> 9.59 mm, vias 2 -> 1
- net /ESC1/VS_C1: track 36.7 -> 29.0 mm
- net /ESC2/VS_A1: track 29.0 -> 21.5 mm
- net /ESC2/VS_C1: track 38.5 -> 31.1 mm
- net Net-(Q303-G): track 18.2 -> 10.9 mm, vias 2 -> 1
- net Net-(Q202-G): track 18.2 -> 11.1 mm, vias 2 -> 1
- net /ESC1/VS_B1: track 29.9 -> 23.5 mm
- net Net-(Q201-G): track 15.7 -> 9.69 mm
- net /ESC2/VS_B1: track 32.9 -> 28.8 mm
- net /ESC1/VS_A1: track 25.6 -> 23.3 mm
- net GND: vias 47 -> 37

Commit message: update lib
Parts:
- removed C147, C163: 10uF/50V, SMTOPT:C_1206
- U201, U301, U401, U501: footprint Package_DFN_QFN:WQFN-28-1EP_4x4mm_P0.4mm_EP2.7x2.7mm -> SMTOPT:WQFN-28-1EP_4x4mm_P0.4mm_EP2.7x2.7mm
- U202, U302, U402, U502: footprint Package_DFN_QFN:QFN-24-1EP_4x4mm_P0.5mm_EP2.7x2.7mm -> SMTOPT:QFN-24-1EP_4x4mm_P0.5mm_EP2.7x2.7mm
- moved Q503 3.11 mm to (126.0, 107.0)
- moved Q401 3.11 mm to (126.0, 123.0)
- moved Q502 3.01 mm to (126.0, 110.2)
- moved Q402 3.01 mm to (126.0, 119.8)
- moved Q501 2.96 mm to (126.0, 113.4)
- moved Q403 2.96 mm to (126.0, 116.6)
- moved C138 2.36 mm to (105.2, 123.0)
- moved C134 2.35 mm to (124.8, 123.0)
- moved C139 2.07 mm to (105.2, 121.0)
- moved C136 2.06 mm to (124.8, 121.0)
- moved C140 1.77 mm to (105.2, 119.0)
- moved C149 1.76 mm to (124.8, 119.0)
- moved C141 1.47 mm to (105.2, 117.0)
- moved C151 1.46 mm to (124.8, 117.0)
- moved C142 1.18 mm to (105.2, 115.0)
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Routing:
- net +3V3: track 89.1 -> 0.00 mm, vias 10 -> 0
- net VCC: track 78.4 -> 0.00 mm, vias 5 -> 0
- net GND: track 52.4 -> 0.00 mm, vias 37 -> 0
- net /ISNS: track 50.8 -> 0.00 mm, vias 3 -> 0
- net /ESC4/VS_C1: track 39.4 -> 0.00 mm, vias 11 -> 0
- net /ESC3/VS_C1: track 38.7 -> 0.00 mm, vias 11 -> 0
- net /SWDIO3: track 36.2 -> 0.00 mm, vias 1 -> 0
- net /SWCLK2: track 35.5 -> 0.00 mm, vias 1 -> 0
- net /SWCLK3: track 32.5 -> 0.00 mm, vias 1 -> 0
- net /DSHOT1: track 31.8 -> 0.00 mm, vias 2 -> 0
- net /ESC3/VS_B1: track 31.4 -> 0.00 mm, vias 11 -> 0
- net /ESC4/VS_B1: track 31.3 -> 0.00 mm, vias 11 -> 0
- net /ESC2/VS_C1: track 31.1 -> 0.00 mm, vias 11 -> 0
- net /SWDIO2: track 30.7 -> 0.00 mm, vias 1 -> 0
- net /ESC1/VS_C1: track 29.0 -> 0.00 mm, vias 11 -> 0
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- removed copper zone on B.Cu, net /ESC1/VS_A1
- removed copper zone on F.Cu, net /ESC1/VS_A1
- removed copper zone on B.Cu, net /ESC1/VS_B1
- removed copper zone on F.Cu, net /ESC1/VS_B1
- removed copper zone on B.Cu, net /ESC1/VS_C1
- removed copper zone on F.Cu, net /ESC1/VS_C1
- removed copper zone on B.Cu, net /ESC2/VS_A1
- removed copper zone on F.Cu, net /ESC2/VS_A1
- removed copper zone on B.Cu, net /ESC2/VS_B1
- removed copper zone on F.Cu, net /ESC2/VS_B1
- removed copper zone on B.Cu, net /ESC2/VS_C1
- removed copper zone on F.Cu, net /ESC2/VS_C1
- removed copper zone on B.Cu, net /ESC3/VS_A1
- removed copper zone on F.Cu, net /ESC3/VS_A1
- removed copper zone on B.Cu, net /ESC3/VS_B1
- removed copper zone on F.Cu, net /ESC3/VS_B1
- removed copper zone on B.Cu, net /ESC3/VS_C1
- removed copper zone on F.Cu, net /ESC3/VS_C1
- removed copper zone on B.Cu, net /ESC4/VS_A1
- removed copper zone on F.Cu, net /ESC4/VS_A1
- removed copper zone on B.Cu, net /ESC4/VS_B1
- removed copper zone on F.Cu, net /ESC4/VS_B1
- removed copper zone on B.Cu, net /ESC4/VS_C1
- removed copper zone on F.Cu, net /ESC4/VS_C1
- removed copper zone on B.Cu, net /LX1
- removed copper zone on B.Cu, net GND
- removed copper zone on F.Cu, net GND
- removed copper zone on In1.Cu, net GND
- removed copper zone on In2.Cu, net GND
- removed copper zone on B.Cu, net GNDPWR
- removed copper zone on F.Cu, net GNDPWR
- removed copper zone on B.Cu, net VBUS
- removed copper zone on F.Cu, net VBUS
- removed copper zone on B.Cu, net VCC
Other:
- board text removed: "+"
- board text removed: "-"
- board text removed: "2025/09/27"
- board text removed: "@DuckWang"
- board text removed: "HW Rev 1.0"
- board text removed: "NekoESC"
- board text removed: "NekoESC AM32 Support"

Commit message: modify hardware
Parts:
- removed C101: 1uF/50V, Capacitor_SMD:C_0603_1608Metric
- removed H101, H102, H103, H104: MountingHole, MountingHole:MountingHole_4.3mm_M4_DIN965
- R107: footprint Resistor_SMD:R_1218_3246Metric -> Resistor_SMD:R_1206_3216Metric
- R217, R218, R219, R220: value 1K -> 10K
- moved R219 48.9 mm to (120.8, 126.7)
- moved R218 37.1 mm to (111.9, 114.9)
- moved R220 36.1 mm to (118.1, 115.3), turned to 180 degrees
- moved R104 17.2 mm to (107.7, 128.1), turned to 180 degrees
- moved U102 15.6 mm to (108.2, 130.6), turned to 90 degrees
- moved U104 12.0 mm to (121.2, 130.6), turned to 0 degrees
- moved C105 11.0 mm to (110.8, 132.6), turned to 0 degrees
- moved L102 7.50 mm to (111.8, 130.3), turned to -90 degrees
- moved C110 5.94 mm to (117.8, 129.6), turned to -90 degrees
- moved C111 5.40 mm to (117.8, 131.4), turned to 90 degrees
- moved R106 3.54 mm to (114.0, 129.5), turned to 90 degrees
- moved R105 3.48 mm to (114.0, 131.4), turned to 90 degrees
- moved R217 3.40 mm to (110.2, 102.4), turned to 180 degrees
- moved C108 2.47 mm to (116.7, 130.1), turned to 90 degrees
- moved J102 1.22 mm to (122.1, 97.4)
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Connections:
- R217 pad 1: /ESC1/BOOT -> +3V3
- R217 pad 2: GND -> /ESC1/NRST
- R218 pad 1: /ESC2/BOOT -> +3V3
- R218 pad 2: GND -> /ESC2/NRST
- R219 pad 1: /ESC3/BOOT -> +3V3
- R219 pad 2: GND -> /ESC3/NRST
- R220 pad 1: /ESC4/BOOT -> +3V3
- R220 pad 2: GND -> /ESC4/NRST
- U201 pad 1: /ESC1/BOOT -> GND
- U301 pad 1: /ESC2/BOOT -> GND
- U401 pad 1: /ESC3/BOOT -> GND
- U501 pad 1: /ESC4/BOOT -> GND
Other:
- board size 38.5 x 38.5 mm -> 32 x 38.5 mm
- board text removed: "BAT GND CUR N C"
- board text removed: "IN1 IN2 IN3 IN4"
- board text removed: "JLCJLCJLCJLC"
