File: NekoESC_V1/NekoESC.kicad_sch (KiCad schematic)
At the start: 62 parts, among them J101 SWD, J102 SWD, J107 JST-SH_8P, U102 ME3121, U103 INA180A1, U104 HT7533-1-SOT89

Commit message: add c1206
Parts:
- C122, C123, C124, C125, C126, C127, C128, C129, C130, C131, C133, C134, C135, C136, C138, C139, C140, C141, C142, C143, C144, C145, C146, C147, C148, C149, C150, C151, C152, C153, C154, C155, C156, C157, C158, C159, C160, C161, C162, C163: footprint Capacitor_SMD:C_1206_3216Metric -> SMTOPT:C_1206
Changed lines of the file:
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@@
 			)
 		)
-		(property "Footprint" "Capacitor_SMD:C_1206_3216Metric"
+		(property "Footprint" "SMTOPT:C_1206"
 			(at 181.3052 48.26 0)
 			(effects
@@
 			)
 		)
-		(property "Footprint" "Capacitor_SMD:C_1206_3216Metric"
+		(property "Footprint" "SMTOPT:C_1206"
 			(at 235.9152 81.28 0)
 			(effects
@@
 			)
 		)
-		(property "Footprint" "Capacitor_SMD:C_1206_3216Metric"
+		(property "Footprint" "SMTOPT:C_1206"
 			(at 251.1552 81.28 0)
 			(effects
@@
 			)
 		)
-		(property "Footprint" "Capacitor_SMD:C_1206_3216Metric"
+		(property "Footprint" "SMTOPT:C_1206"
 			(at 266.3952 81.28 0)
 			(effects
@@
 			)
 		)
-		(property "Footprint" "Capacitor_SMD:C_1206_3216Metric"
+		(property "Footprint" "SMTOPT:C_1206"
 			(at 196.5452 48.26 0)
 			(effects
@@
 			)
 		)
-		(property "Footprint" "Capacitor_SMD:C_1206_3216Metric"
+		(property "Footprint" "SMTOPT:C_1206"
 			(at 206.7052 81.28 0)
 			(effects
@@
 			)
 		)
-		(property "Footprint" "Capacitor_SMD:C_1206_3216Metric"
+		(property "Footprint" "SMTOPT:C_1206"
 			(at 225.7552 48.26 0)
 			(effects
@@
 			)
 		)
-		(property "Footprint" "Capacitor_SMD:C_1206_3216Metric"
+		(property "Footprint" "SMTOPT:C_1206"
 			(at 240.9952 81.28 0)
 			(effects
@@
 			)
 		)
-		(property "Footprint" "Capacitor_SMD:C_1206_3216Metric"
+		(property "Footprint" "SMTOPT:C_1206"
 			(at 271.4752 81.28 0)
 			(effects
@@
 			)
 		)
-		(property "Footprint" "Capacitor_SMD:C_1206_3216Metric"
+		(property "Footprint" "SMTOPT:C_1206"
 			(at 230.8352 81.28 0)
 			(effects
@@
 			)
 		)
-		(property "Footprint" "Capacitor_SMD:C_1206_3216Metric"
+		(property "Footprint" "SMTOPT:C_1206"
 			(at 225.7552 81.28 0)
 			(effects
@@
 			)
 		)
-		(property "Footprint" "Capacitor_SMD:C_1206_3216Metric"
+		(property "Footprint" "SMTOPT:C_1206"
 			(at 206.7052 48.26 0)
 			(effects
@@
 			)
 		)
-		(property "Footprint" "Capacitor_SMD:C_1206_3216Metric"
+		(property "Footprint" "SMTOPT:C_1206"
 			(at 201.6252 48.26 0)
 			(effects
@@
 			)
 		)
-		(property "Footprint" "Capacitor_SMD:C_1206_3216Metric"
+		(property "Footprint" "SMTOPT:C_1206"
 			(at 191.4652 48.26 0)
 			(effects
@@
 			)
 		)
-		(property "Footprint" "Capacitor_SMD:C_1206_3216Metric"
+		(property "Footprint" "SMTOPT:C_1206"
 			(at 176.2252 81.28 0)
 			(effects
@@
 			)
 		)
-		(property "Footprint" "Capacitor_SMD:C_1206_3216Metric"
+		(property "Footprint" "SMTOPT:C_1206"
 			(at 271.4752 48.26 0)
 			(effects
@@
 			)
 		)
-		(property "Footprint" "Capacitor_SMD:C_1206_3216Metric"
+		(property "Footprint" "SMTOPT:C_1206"
 			(at 166.0652 81.28 0)
 			(effects
@@
 			)
 		)
-		(property "Footprint" "Capacitor_SMD:C_1206_3216Metric"
+		(property "Footprint" "SMTOPT:C_1206"
 			(at 171.1452 81.28 0)
 			(effects
@@
 			)
 		)
-		(property "Footprint" "Capacitor_SMD:C_1206_3216Metric"
+		(property "Footprint" "SMTOPT:C_1206"
 			(at 176.2252 48.26 0)
 			(effects
@@
 			)
 		)
-		(property "Footprint" "Capacitor_SMD:C_1206_3216Metric"
+		(property "Footprint" "SMTOPT:C_1206"
 			(at 201.6252 81.28 0)
 			(effects
@@
 			)
 		)
-		(property "Footprint" "Capacitor_SMD:C_1206_3216Metric"
+		(property "Footprint" "SMTOPT:C_1206"
 			(at 266.3952 48.26 0)
 			(effects
@@
 			)
 		)
-		(property "Footprint" "Capacitor_SMD:C_1206_3216Metric"
+		(property "Footprint" "SMTOPT:C_1206"
 			(at 186.3852 81.28 0)
 			(effects
@@
 			)
 		)
-		(property "Footprint" "Capacitor_SMD:C_1206_3216Metric"
+		(property "Footprint" "SMTOPT:C_1206"
 			(at 246.0752 81.28 0)
 			(effects
@@
 			)
 		)
-		(property "Footprint" "Capacitor_SMD:C_1206_3216Metric"
+		(property "Footprint" "SMTOPT:C_1206"
 			(at 160.9852 81.28 0)
 			(effects
@@
 			)
 		)
-		(property "Footprint" "Capacitor_SMD:C_1206_3216Metric"
+		(property "Footprint" "SMTOPT:C_1206"
 			(at 171.1452 48.26 0)
 			(effects
@@
 			)
 		)
-		(property "Footprint" "Capacitor_SMD:C_1206_3216Metric"
+		(property "Footprint" "SMTOPT:C_1206"
 			(at 251.1552 48.26 0)
 			(effects
@@
 			)
 		)
-		(property "Footprint" "Capacitor_SMD:C_1206_3216Metric"
+		(property "Footprint" "SMTOPT:C_1206"
 			(at 191.4652 81.28 0)
 			(effects
@@
 			)
 		)
-		(property "Footprint" "Capacitor_SMD:C_1206_3216Metric"
+		(property "Footprint" "SMTOPT:C_1206"
 			(at 261.3152 81.28 0)
 			(effects
@@
 			)
 		)
-		(property "Footprint" "Capacitor_SMD:C_1206_3216Metric"
+		(property "Footprint" "SMTOPT:C_1206"
 			(at 186.3852 48.26 0)
 			(effects
@@
 			)
 		)
-		(property "Footprint" "Capacitor_SMD:C_1206_3216Metric"
+		(property "Footprint" "SMTOPT:C_1206"
 			(at 160.9852 48.26 0)
 			(effects
@@
 			)
 		)
-		(property "Footprint" "Capacitor_SMD:C_1206_3216Metric"
+		(property "Footprint" "SMTOPT:C_1206"
 			(at 246.0752 48.26 0)
 			(effects
@@
 			)
 		)
-		(property "Footprint" "Capacitor_SMD:C_1206_3216Metric"
+		(property "Footprint" "SMTOPT:C_1206"
 			(at 230.8352 48.26 0)
 			(effects
@@
 			)
 		)
-		(property "Footprint" "Capacitor_SMD:C_1206_3216Metric"
+		(property "Footprint" "SMTOPT:C_1206"
 			(at 240.9952 48.26 0)
 			(effects
@@
 			)
 		)
-		(property "Footprint" "Capacitor_SMD:C_1206_3216Metric"
+		(property "Footprint" "SMTOPT:C_1206"
 			(at 261.3152 48.26 0)
 			(effects
@@
 			)
 		)
-		(property "Footprint" "Capacitor_SMD:C_1206_3216Metric"
+		(property "Footprint" "SMTOPT:C_1206"
 			(at 256.2352 81.28 0)
 			(effects
@@
 			)
 		)
-		(property "Footprint" "Capacitor_SMD:C_1206_3216Metric"
+		(property "Footprint" "SMTOPT:C_1206"
 			(at 235.9152 48.26 0)
 			(effects
@@
 			)
 		)
-		(property "Footprint" "Capacitor_SMD:C_1206_3216Metric"
+		(property "Footprint" "SMTOPT:C_1206"
 			(at 196.5452 81.28 0)
 			(effects
@@
 			)
 		)
-		(property "Footprint" "Capacitor_SMD:C_1206_3216Metric"
+		(property "Footprint" "SMTOPT:C_1206"
 			(at 166.0652 48.26 0)
 			(effects
@@
 			)
 		)
-		(property "Footprint" "Capacitor_SMD:C_1206_3216Metric"
+		(property "Footprint" "SMTOPT:C_1206"
 			(at 181.3052 81.28 0)
 			(effects
@@
 			)
 		)
-		(property "Footprint" "Capacitor_SMD:C_1206_3216Metric"
+		(property "Footprint" "SMTOPT:C_1206"
 			(at 256.2352 48.26 0)
 			(effects

Commit message: update lib
Parts:
- removed C122, C123, C124, C125, C126, C127, C128, C129, C130, C131, C133, C135, C147, C148, C150, C152, C154, C156, C158, C160, C162, C163: 10uF/50V, SMTOPT:C_1206, symbol Device:C

Commit message: modify hardware
Parts:
- removed C101: 1uF/50V, Capacitor_SMD:C_0603_1608Metric, symbol Device:C
- removed H101, H102, H103, H104: MountingHole, MountingHole:MountingHole_4.3mm_M4_DIN965, symbol Mechanical:MountingHole
- R107: footprint Resistor_SMD:R_1218_3246Metric -> Resistor_SMD:R_1206_3216Metric
